File: placafrontal(sensores)/placafrontal(sensores).kicad_pcb (KiCad board)
At the start: 2 copper layers, 17 parts, among them J1 Conn_01x06_Female, U1 CNY70, U2 CNY70, U3 CNY70, U4 CNY70, U5 CNY70, U6 CNY70, U7 4053

Commit message: 1.1
Parts:
- added REF**: MountingHole_2.2mm_M2, MountingHole:MountingHole_2.2mm_M2, F.Cu at (181.6, 82.5)
- added REF**: MountingHole_2.2mm_M2, MountingHole:MountingHole_2.2mm_M2, F.Cu at (199.4, 82.5)
- U7: footprint Package_DIP:DIP-10_W7.62mm_LongPads -> Package_DIP:DIP-16_W7.62mm_LongPads
- moved U6 97.1 mm to (210.8, 55.9)
- moved R9 84.6 mm to (212.3, 52.1)
- moved U7 82.9 mm to (199.4, 66.0), turned to 270 degrees
- moved R7 79.9 mm to (203.2, 52.1)
- moved U5 77.4 mm to (201.9, 55.9)
- moved R6 70.6 mm to (212.1, 62.2)
- moved R8 70.2 mm to (194.3, 62.2)
- moved R4 69.3 mm to (185.7, 52.1)
- moved J1 64.0 mm to (193.0, 77.5), turned to 270 degrees
- moved U4 62.9 mm to (193.0, 55.9)
- moved R5 61.6 mm to (203.2, 62.2)
- moved R2 58.9 mm to (176.5, 62.2)
- moved R3 56.0 mm to (185.7, 62.2)
- moved R1 50.6 mm to (167.6, 62.2)
- moved U3 47.9 mm to (184.2, 55.9)
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Connections:
- J1 pad 6: /linea_select -> /linea_selec
Routing:
- net +5V: track 0.00 -> 96.0 mm, vias 0 -> 1
- net GND: track 0.00 -> 90.3 mm, vias 0 -> 1
- net /sensor6: track 0.00 -> 33.3 mm
- net /sensor3: track 0.00 -> 31.9 mm, vias 0 -> 3
- net /sensor1: track 0.00 -> 29.8 mm, vias 0 -> 1
- net /sensor2: track 0.00 -> 28.3 mm, vias 0 -> 1
- net /sensor5: track 0.00 -> 27.0 mm, vias 0 -> 1
- net /sensor4: track 0.00 -> 23.3 mm, vias 0 -> 1
- net /linea2: track 0.00 -> 19.8 mm
- net /linea3: track 0.00 -> 19.3 mm
- net /linea_selec: track 0.00 -> 11.4 mm
- net Net-(R4-Pad1): track 0.00 -> 9.40 mm
- net Net-(R1-Pad2): track 0.00 -> 8.97 mm
- net Net-(R7-Pad2): track 0.00 -> 8.17 mm
- net Net-(R4-Pad2): track 0.00 -> 7.93 mm
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Other:
- board outline added: 54.6 x 35.6 mm
- board text added: "5V"
- board text added: "GND"
- board text added: "L1"
