File: placafrontal(sensores)/placafrontal(sensores).sch (KiCad schematic (older format))
At the start: 17 parts, among them J1 Conn_01x06_Female, U1 CNY70, U2 CNY70, U3 CNY70, U4 CNY70, U5 CNY70, U6 CNY70, U7 4053

Commit message: 1.1
Parts:
- U7: footprint Package_DIP:DIP-10_W7.62mm_LongPads -> Package_DIP:DIP-16_W7.62mm_LongPads
Changed lines of the file:
@@
 EESchema Schematic File Version 4
+LIBS:placafrontal(sensores)-cache
 EELAYER 26 0
 EELAYER END
@@
 F 0 "U7" H 8550 4628 50  0000 C CNN
 F 1 "4053" H 8550 4537 50  0000 C CNN
-F 2 "Package_DIP:DIP-10_W7.62mm_LongPads" H 8550 3550 50  0001 C CNN
+F 2 "Package_DIP:DIP-16_W7.62mm_LongPads" H 8550 3550 50  0001 C CNN
 F 3 "http://www.intersil.com/content/dam/Intersil/documents/cd40/cd4051bms-52bms-53bms.pdf" H 8550 3550 50  0001 C CNN
 	1    8550 3550
